File: Leiterplatte/VQC10x4_ohne_Controller_V3.kicad_sch (KiCad schematic)
At the start: 34 parts, among them J2 Conn_02x10_Odd_Even, J3 Conn_02x10_Odd_Even, Q1 BD140, Q2 BD140, Q3 BD140, Q4 BD140, Q5 BD140, Q6 BD140, Q7 BD140, U1 74HCT138, U2 74LS154, U3 74LS123

Commit message: UPD: Neue Leiterplattenversion
Parts:
- removed D1, D2, D3, D4: VQC 10, DDR-RFT:VQC10, symbol DDR_Library:VQC10
- removed U2: 74LS154, Package_DIP:DIP-24_W15.24mm_LongPads, symbol 74xx:74LS154
- added H5, H6, H7, H8: VQC 10, DDR_RFT_KiCAD_Library:VQC10, symbol DDR_Library:VQC10
- added JP3, JP4: Jumper_2_Bridged, TestPoint:TestPoint_2Pads_Pitch2.54mm_Drill0.8mm, symbol Jumper:Jumper_2_Bridged
- added U2, U3: 74HCT138, Package_DIP:DIP-16_W7.62mm_LongPads, symbol 74xx:74HCT138
- C2: value 100µ -> C_Polarized
- C3: value 100n -> C
- D1: renamed from D5; value 1N4148 -> SAY40; footprint Diode_THT:D_A-405_P2.54mm_Vertical_AnodeUp -> Diode_THT:D_A-405_P7.62mm_Horizontal
- J1: renamed from J2; footprint Connector_PinHeader_2.54mm:PinHeader_2x10_P2.54mm_Horizontal -> Connector_IDC:IDC-Header_2x10_P2.54mm_Horizontal
- J2: renamed from J3; footprint Connector_PinHeader_2.54mm:PinHeader_2x10_P2.54mm_Horizontal -> Connector_IDC:IDC-Header_2x10_P2.54mm_Horizontal
- R1, R2, R3, R4, R5, R6, R7: footprint Resistor_THT:R_Axial_DIN0204_L3.6mm_D1.6mm_P5.08mm_Vertical -> Resistor_THT:R_Axial_DIN0204_L3.6mm_D1.6mm_P5.08mm_Horizontal
- renumbered U3 to U4
Connections:
- net +5V: now also H5.14 (Ucc), H6.14 (Ucc), H7.14 (Ucc), H8.14 (Ucc), U2.16 (VCC), U2.6 (E2), U3.16 (VCC)
- net D1: now also H5.1 (D1), H6.1 (D1), H7.1 (D1), H8.1 (D1)
- net D2: now also H5.8 (D2), H6.8 (D2), H7.8 (D2), H8.8 (D2)
- net D3: now also H5.4 (D3), H6.4 (D3), H7.4 (D3), H8.4 (D3)
- net D4: now also H5.11 (D4), H6.11 (D4), H7.11 (D4), H8.11 (D4)
- net D5: now also H5.15 (D5), H6.15 (D5), H7.15 (D5), H8.15 (D5)
- net GND: now also U4.10 (B), U4.11 (Clr), U4.9 (A), H5.10 (Cool), H5.13 (Cool), H5.16 (GND), H5.24 (GND), H5.3 (Cool), H5.6 (Cool), H6.10 (Cool), H6.13 (Cool), H6.16 (GND), H6.24 (GND), H6.3 (Cool), H6.6 (Cool), H7.10 (Cool), H7.13 (Cool), H7.16 (GND), H7.24 (GND), H7.3 (Cool), H7.6 (Cool), H8.10 (Cool), H8.13 (Cool), H8.16 (GND), H8.24 (GND), H8.3 (Cool), H8.6 (Cool), U2.8 (GND), U3.8 (GND); no longer J1.17 (Pin_17), J2.17 (Pin_17)
- net S0: now also H5.2 (CP1), U2.15 (~{Y0})
- net S1: now also H5.5 (CP2), U2.14 (~{Y1})
- net S10: now also H7.9 (CP3), U3.13 (~{Y2})
- net S11: now also H7.12 (CP4), U3.12 (~{Y3})
- net S12: now also H8.2 (CP1), U3.11 (~{Y4})
- net S13: now also H8.5 (CP2), U3.10 (~{Y5})
- net S14: now also H8.9 (CP3), U3.9 (~{Y6})
- net S15: now also H8.12 (CP4), U3.7 (~{Y7})
- net S2: now also H5.9 (CP3), U2.13 (~{Y2})
- net S3: now also H5.12 (CP4), U2.12 (~{Y3})
- net S4: now also H6.2 (CP1), U2.11 (~{Y4})
- net S5: now also H6.5 (CP2), U2.10 (~{Y5})
- net S6: now also H6.9 (CP3), U2.9 (~{Y6})
- net S7: now also H6.12 (CP4), U2.7 (~{Y7})
- net S8: now also H7.2 (CP1), U3.15 (~{Y0})
- net S9: now also H7.5 (CP2), U3.14 (~{Y1})
- net SD0: now also U2.1 (A0), U3.1 (A0)
- net SD1: now also U2.2 (A1), U3.2 (A1)
- net SD2: now also U2.3 (A2), U3.3 (A2)
- net SD3: now also U2.4 (~{E0}), U3.6 (E2)
- net SD4: now also JP1.1 (A); no longer JP2.1 (A)
- net SD5: now also JP2.1 (A); no longer JP1.1 (A)
- net SD6: now also JP3.1 (A)
- net Z1: now also H5.20 (Z1), H6.20 (Z1), H7.20 (Z1), H8.20 (Z1)
- net Z2: now also H5.21 (Z2), H6.21 (Z2), H7.21 (Z2), H8.21 (Z2)
- net Z3: now also H5.19 (Z3), H6.19 (Z3), H7.19 (Z3), H8.19 (Z3)
- net Z4: now also H5.22 (Z4), H6.22 (Z4), H7.22 (Z4), H8.22 (Z4)
- net Z5: now also H5.23 (Z5), H6.23 (Z5), H7.23 (Z5), H8.23 (Z5)
- net Z6: now also H5.18 (Z6), H6.18 (Z6), H7.18 (Z6), H8.18 (Z6)
- net Z7: now also H5.17 (Z7), H6.17 (Z7), H7.17 (Z7), H8.17 (Z7)
- net at JP2.2 (B): now also JP1.2 (B), JP3.2 (B), JP4.2 (B), U2.5 (~{E1}), U3.4 (~{E0}), U3.5 (~{E1})
- new net SD7: J1.17 (Pin_17), J2.17 (Pin_17), JP4.1 (A)
- no-connect marks 9 -> 6
Other:
- title: 8x VQC10 ohne Controller -> 4x VQC10 ohne Controller
- moved on the sheet: C2, U1, U4B, U4C
